Commit message: update hokuyo position
changing z position of hokuyo to match with the turtlebot in urdf and sdf.

File: models/turtlebot/model.urdf (robot description, URDF)
Before this commit: robot turtlebot, 5 links, 4 joints
Joints:
- joint turtlebot__hokuyo_joint: origin xyz=0       0       1.03499 rpy=0  0  0 -> xyz=0       0       0.45 rpy=0  0  0

Commit message: urdf to support RVIZ
modified URDF to show turtlebot in RVIZ

File: models/turtlebot/model.urdf (robot description, URDF)
Before this commit: robot turtlebot, 5 links, 4 joints
Links:
- link turtlebot/create::base: geometry collision cylinder length=0.061163 radius=0.016495; collision sphere radius=0.015000
- link turtlebot/hokuyo::link: geometry collision box size=0.05 0.05 0.041; collision cylinder length=0.029 radius=0.021
- link turtlebot__rack: geometry collision box size=0.233502 0.314845 0.006401; collision box size=0.288000 0.315000 0.006401
Joints:
- joint turtlebot__create__left_wheel: limit lower=0.0 upper=0.0 effort=0.0 velocity=0.0 -> lower=0 upper=0 effort=0 velocity=0
- joint turtlebot__create__right_wheel: limit lower=0.0 upper=0.0 effort=0.0 velocity=0.0 -> lower=0 upper=0 effort=0 velocity=0
- joint turtlebot__hokuyo_joint: origin xyz=0       0       0.45 rpy=0  0  0 -> xyz=0     0     0.485 rpy=0  0  0
